File: nimh-charger.kicad_sch (KiCad schematic)
At the start: 25 parts, among them J1 PWR_IN

Commit message: Final tweaks and silk
Parts:
- added TP1: 5V, Connector_Wire:SolderWire-0.5sqmm_1x01_D0.9mm_OD2.1mm_Relief, symbol Connector:TestPoint
- added TP2: GND, Connector_Wire:SolderWire-0.5sqmm_1x01_D0.9mm_OD2.1mm_Relief, symbol Connector:TestPoint
Connections:
- net +5V: now also TP1.1
- net GND: now also TP2.1
Changed lines of the file:
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@@
     (pin "2")
+  )
+  (symbol (lib_id "power:GND") (at 59.69 73.66 0) (unit 1)
+    (in_bom yes) (on_board yes) (fields_autoplaced)
+    (property "Reference" "#PWR014" (id 0) (at 59.69 80.01 0)
+      (effects (font (size 1.27 1.27)) hide)
+    )
+    (property "Value" "GND" (id 1) (at 59.69 78.1034 0))
+    (property "Footprint" "" (id 2) (at 59.69 73.66 0)
+      (effects (font (size 1.27 1.27)) hide)
+    )
+    (property "Datasheet" "" (id 3) (at 59.69 73.66 0)
+      (effects (font (size 1.27 1.27)) hide)
+    )
+    (pin "1")
   )
   (symbol (lib_id "Device:R_Small") (at 67.31 46.99 0) (unit 1)
@@
     )
   )
+  (symbol (lib_id "Connector:TestPoint") (at 59.69 73.66 0) (unit 1)
+    (in_bom yes) (on_board yes)
+    (property "Reference" "TP2" (id 0) (at 61.087 69.5233 0)
+      (effects (font (size 1.27 1.27)) (justify left))
+    )
+    (property "Value" "GND" (id 1) (at 61.087 72.0602 0)
+      (effects (font (size 1.27 1.27)) (justify left))
+    )
+    (property "Footprint" "Connector_Wire:SolderWire-0.5sqmm_1x01_D0.9mm_OD2.1mm_Relief" (id 2) (at 64.77 73.66 0)
+      (effects (font (size 1.27 1.27)) hide)
+    )
+    (property "Datasheet" "~" (id 3) (at 64.77 73.66 0)
+      (effects (font (size 1.27 1.27)) hide)
+    )
+    (pin "1")
+  )
   (symbol (lib_id "Device:R_Small") (at 59.69 44.45 0) (mirror x) (unit 1)
     (in_bom yes) (on_board yes) (fields_autoplaced)
@@
     (pin "1")
     (pin "2")
+  )
+  (symbol (lib_id "Connector:TestPoint") (at 52.07 73.66 180) (unit 1)
+    (in_bom yes) (on_board yes) (fields_autoplaced)
+    (property "Reference" "TP1" (id 0) (at 53.467 76.1273 0)
+      (effects (font (size 1.27 1.27)) (justify right))
+    )
+    (property "Value" "5V" (id 1) (at 53.467 78.6642 0)
+      (effects (font (size 1.27 1.27)) (justify right))
+    )
+    (property "Footprint" "Connector_Wire:SolderWire-0.5sqmm_1x01_D0.9mm_OD2.1mm_Relief" (id 2) (at 46.99 73.66 0)
+      (effects (font (size 1.27 1.27)) hide)
+    )
+    (property "Datasheet" "~" (id 3) (at 46.99 73.66 0)
+      (effects (font (size 1.27 1.27)) hide)
+    )
+    (pin "1")
   )
   (symbol (lib_id "power:GND") (at 63.5 57.15 0) (unit 1)
@@
     (pin "2")
   )
+  (symbol (lib_id "power:+5V") (at 52.07 73.66 0) (unit 1)
+    (in_bom yes) (on_board yes) (fields_autoplaced)
+    (property "Reference" "#PWR013" (id 0) (at 52.07 77.47 0)
+      (effects (font (size 1.27 1.27)) hide)
+    )
+    (property "Value" "+5V" (id 1) (at 52.07 70.0842 0))
+    (property "Footprint" "" (id 2) (at 52.07 73.66 0)
+      (effects (font (size 1.27 1.27)) hide)
+    )
+    (property "Datasheet" "" (id 3) (at 52.07 73.66 0)
+      (effects (font (size 1.27 1.27)) hide)
+    )
+    (pin "1")
+  )
   (symbol (lib_id "power:+5V") (at 44.45 33.02 0) (unit 1)
     (in_bom yes) (on_board yes) (fields_autoplaced)
@@
       (reference "#PWR012") (unit 1) (value "GND") (footprint "")
     )
+    (path "/cb12900c-7283-41cb-be2d-8d63952851e7"
+      (reference "#PWR013") (unit 1) (value "+5V") (footprint "")
+    )
+    (path "/445391b4-eb4c-47dc-9769-1479ed41a761"
+      (reference "#PWR014") (unit 1) (value "GND") (footprint "")
+    )
     (path "/0d7ea15c-2362-4fab-90f8-243454047248"
       (reference "BT1") (unit 1) (value "Battery_Cell") (footprint "Battery:BatteryHolder_Keystone_2460_1xAA")
@@
       (reference "R9") (unit 1) (value "120R") (footprint "Resistor_THT:R_Axial_DIN0309_L9.0mm_D3.2mm_P12.70mm_Horizontal")
     )
-  )
+    (path "/9dfad586-c5b6-4d25-b1ad-e1b0b6cec690"
+      (reference "TP1") (unit 1) (value "5V") (footprint "Connector_Wire:SolderWire-0.5sqmm_1x01_D0.9mm_OD2.1mm_Relief")
+    )
+    (path "/82e86ded-6ef0-4071-9932-633313c36400"
+      (reference "TP2") (unit 1) (value "GND") (footprint "Connector_Wire:SolderWire-0.5sqmm_1x01_D0.9mm_OD2.1mm_Relief")
+    )
+  )

Commit message: Added LCSC part numbers and ibom
Parts:
- BT1, BT2, BT3, BT4, H1, H2, TP1, TP2: LCSC (none) -> -
- D1, D6, D7, D8, D9: LCSC (none) -> C417347
- D2, D3, D4, D5: LCSC (none) -> C898870
- R1: LCSC (none) -> C2896818
- R2, R3, R4, R5, R6, R7, R8, R9: LCSC (none) -> C119306
Changed lines of the file:
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@@
+      (effects (font (size 1.27 1.27)) hide)
+    )
+    (property "LCSC" "-" (id 4) (at 114.3 54.61 0)
       (effects (font (size 1.27 1.27)) hide)
     )
@@
     )
     (property "Datasheet" "~" (id 3) (at 110.49 44.45 0)
+      (effects (font (size 1.27 1.27)) hide)
+    )
+    (property "LCSC" "C119306" (id 4) (at 110.49 44.45 0)
       (effects (font (size 1.27 1.27)) hide)
     )
@@
       (effects (font (size 1.27 1.27)) hide)
     )
+    (property "LCSC" "-" (id 4) (at 63.5 54.61 0)
+      (effects (font (size 1.27 1.27)) hide)
+    )
     (pin "1")
     (pin "2")
@@
       (effects (font (size 1.27 1.27)) hide)
     )
+    (property "LCSC" "C119306" (id 4) (at 118.11 46.99 0)
+      (effects (font (size 1.27 1.27)) hide)
+    )
     (pin "1")
     (pin "2")
@@
       (effects (font (size 1.27 1.27)) hide)
     )
+    (property "LCSC" "C119306" (id 4) (at 85.09 44.45 0)
+      (effects (font (size 1.27 1.27)) hide)
+    )
     (pin "1")
     (pin "2")
@@
     )
     (property "Datasheet" "~" (id 3) (at 139.7 53.086 90)
+      (effects (font (size 1.27 1.27)) hide)
+    )
+    (property "LCSC" "-" (id 4) (at 139.7 54.61 0)
       (effects (font (size 1.27 1.27)) hide)
     )
@@
       (effects (font (size 1.27 1.27)) hide)
     )
+    (property "LCSC" "C898870" (id 4) (at 88.9 35.56 0)
+      (effects (font (size 1.27 1.27)) hide)
+    )
     (pin "1")
     (pin "2")
@@
       (effects (font (size 1.27 1.27)) hide)
     )
+    (property "LCSC" "C119306" (id 4) (at 143.51 46.99 0)
+      (effects (font (size 1.27 1.27)) hide)
+    )
     (pin "1")
     (pin "2")
@@
     )
     (property "Datasheet" "~" (id 3) (at 67.31 46.99 0)
+      (effects (font (size 1.27 1.27)) hide)
+    )
+    (property "LCSC" "C119306" (id 4) (at 67.31 46.99 0)
       (effects (font (size 1.27 1.27)) hide)
     )
@@
       (effects (font (size 1.27 1.27)) hide)
     )
+    (property "LCSC" "C898870" (id 4) (at 63.5 35.56 0)
+      (effects (font (size 1.27 1.27)) hide)
+    )
     (pin "1")
     (pin "2")
@@
       (effects (font (size 1.27 1.27)) hide)
     )
+    (property "LCSC" "-" (id 4) (at 88.9 54.61 0)
+      (effects (font (size 1.27 1.27)) hide)
+    )
     (pin "1")
     (pin "2")
@@
     )
     (property "Datasheet" "~" (id 3) (at 25.4 81.28 0)
+      (effects (font (size 1.27 1.27)) hide)
+    )
+    (property "LCSC" "-" (id 4) (at 25.4 81.28 0)
       (effects (font (size 1.27 1.27)) hide)
     )
@@
       (effects (font (size 1.27 1.27)) hide)
     )
+    (property "LCSC" "C898870" (id 4) (at 139.7 35.56 0)
+      (effects (font (size 1.27 1.27)) hide)
+    )
     (pin "1")
     (pin "2")
@@
     )
     (property "Datasheet" "~" (id 3) (at 25.4 76.2 0)
+      (effects (font (size 1.27 1.27)) hide)
+    )
+    (property "LCSC" "-" (id 4) (at 25.4 76.2 0)
       (effects (font (size 1.27 1.27)) hide)
     )
@@
       (effects (font (size 1.27 1.27)) hide)
     )
+    (property "LCSC" "-" (id 4) (at 59.69 73.66 0)
+      (effects (font (size 1.27 1.27)) hide)
+    )
     (pin "1")
   )
@@
       (effects (font (size 1.27 1.27)) hide)
     )
+    (property "LCSC" "C119306" (id 4) (at 59.69 44.45 0)
+      (effects (font (size 1.27 1.27)) hide)
+    )
     (pin "1")
     (pin "2")
@@
     )
     (property "Datasheet" "~" (id 3) (at 67.31 41.91 90)
+      (effects (font (size 1.27 1.27)) hide)
+    )
+    (property "LCSC" "C417347" (id 4) (at 67.31 41.91 0)
       (effects (font (size 1.27 1.27)) hide)
     )
@@
       (effects (font (size 1.27 1.27)) hide)
     )
+    (property "LCSC" "C417347" (id 4) (at 118.11 41.91 0)
+      (effects (font (size 1.27 1.27)) hide)
+    )
     (pin "1")
     (pin "2")
@@
       (effects (font (size 1.27 1.27)) hide)
     )
+    (property "LCSC" "C119306" (id 4) (at 135.89 44.45 0)
+      (effects (font (size 1.27 1.27)) hide)
+    )
     (pin "1")
     (pin "2")
@@
     )
     (property "Datasheet" "~" (id 3) (at 46.99 73.66 0)
+      (effects (font (size 1.27 1.27)) hide)
+    )
+    (property "LCSC" "-" (id 4) (at 52.07 73.66 0)
       (effects (font (size 1.27 1.27)) hide)
     )
@@
       (effects (font (size 1.27 1.27)) hide)
     )
+    (property "LCSC" "C417347" (id 4) (at 92.71 41.91 0)
+      (effects (font (size 1.27 1.27)) hide)
+    )
     (pin "1")
     (pin "2")
@@
     )
     (property "Datasheet" "~" (id 3) (at 44.45 40.64 0)
+      (effects (font (size 1.27 1.27)) hide)
+    )
+    (property "LCSC" "C2896818" (id 4) (at 44.45 40.64 0)
       (effects (font (size 1.27 1.27)) hide)
     )
@@
       (effects (font (size 1.27 1.27)) hide)
     )
+    (property "LCSC" "C898870" (id 4) (at 114.3 35.56 0)
+      (effects (font (size 1.27 1.27)) hide)
+    )
     (pin "1")
     (pin "2")
@@
       (effects (font (size 1.27 1.27)) hide)
     )
+    (property "LCSC" "C417347" (id 4) (at 143.51 41.91 0)
+      (effects (font (size 1.27 1.27)) hide)
+    )
     (pin "1")
     (pin "2")
@@
       (effects (font (size 1.27 1.27)) hide)
     )
+    (property "LCSC" "C417347" (id 4) (at 44.45 35.56 0)
+      (effects (font (size 1.27 1.27)) hide)
+    )
     (pin "1")
     (pin "2")
@@
       (effects (font (size 1.27 1.27)) hide)
     )
+    (property "LCSC" "C119306" (id 4) (at 92.71 46.99 0)
+      (effects (font (size 1.27 1.27)) hide)
+    )

Commit message: SMD 2-cell chaining version
Parts:
- removed BT3, BT4: Battery_Cell, Battery:BatteryHolder_Keystone_2460_1xAA, symbol Device:Battery_Cell
- removed D4, D5: 1N400X, Diode_THT:D_DO-41_SOD81_P12.70mm_Horizontal, symbol Device:D_Small
- removed D8: CH3, LED_THT:LED_D5.0mm, symbol Device:LED_Small
- removed D9: CH4, LED_THT:LED_D5.0mm, symbol Device:LED_Small
- removed R4, R5, R8, R9: 120R, Resistor_THT:R_Axial_DIN0309_L9.0mm_D3.2mm_P12.70mm_Horizontal, symbol Device:R_Small
- added H3, H4: MountingHole, MountingHole:MountingHole_3.2mm_M3_DIN965, symbol Mechanical:MountingHole
- added TP3: 5V, TestPoint:TestPoint_Pad_2.5x2.5mm, symbol Connector:TestPoint
- added TP4: GND, TestPoint:TestPoint_Pad_2.5x2.5mm, symbol Connector:TestPoint
- BT1, BT2: footprint Battery:BatteryHolder_Keystone_2460_1xAA -> nimh-charger:BatteryHolder_Keystone_2460_1xAA
- D1, D6, D7: footprint LED_THT:LED_D5.0mm -> LED_SMD:LED_0805_2012Metric; LCSC C417347 -> C965812
- D2, D3: footprint Diode_THT:D_DO-41_SOD81_P12.70mm_Horizontal -> Diode_SMD:D_SMA; LCSC C898870 -> C2892325
- J1: footprint nimh-charger:KH-TYPE-C-2P -> Connector_USB:USB_Micro-B_Molex-105017-0001; symbol nimh-charger:USB_C_power_only -> Connector:USB_B_Micro; LCSC C2919656 -> C136000
- R1: value 470R -> 1k; footprint Resistor_THT:R_Axial_DIN0309_L9.0mm_D3.2mm_P12.70mm_Horizontal -> Resistor_SMD:R_0805_2012Metric; LCSC C2896818 -> (none)
- R2, R3, R6, R7: footprint Resistor_THT:R_Axial_DIN0309_L9.0mm_D3.2mm_P12.70mm_Horizontal -> Resistor_SMD:R_0805_2012Metric; LCSC C119306 -> (none)
- TP1, TP2: footprint Connector_Wire:SolderWire-0.5sqmm_1x01_D0.9mm_OD2.1mm_Relief -> TestPoint:TestPoint_Pad_2.5x2.5mm
Connections:
- net +5V: now also TP3.1
- net GND: now also J1.5 (GND), TP4.1; no longer J1.2 (GND)
- no-connect marks 1 -> 4
